Commit message: Step 53 Differential Drive Plugin completed

File: install/robot_description_pkg/share/robot_description_pkg/urdf/mobile_robot.urdf (robot description, URDF)
Before this commit: robot mobile_robot, 7 links, 6 joints
Joints:
- joint left_wheel_joint: axis (none) -> 0 1 0; type fixed -> continuous
- joint right_wheel_joint: axis (none) -> 0 1 0; type fixed -> continuous
